File: BlampKnob.kicad_pcb (KiCad board)
At the start: 2 copper layers, 15.2 x 25.4 mm, 12 parts, among them J1 S5B-PH-K-S, SW1 PEC11H-4220F-S0024

Commit message: Add BoardInfo footprint and project variables, B_TITLE, B_REV, and B_COMPANY
Parts:
- added REF**: BoardInfo, VZ_Library:BoardInfo, B.Cu at (166.4, 96.2)
