File: BlampKnob.kicad_sch (KiCad schematic)
At the start: 12 parts, among them J1 S5B-PH-K-S, SW1 PEC11H-4220F-S0024

Commit message: Add BoardInfo footprint and project variables, B_TITLE, B_REV, and B_COMPANY
Other:
- company: VZ -> ${B_COMPANY}
- title: Blamp Knob -> ${B_TITLE}
Changed lines of the file:
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@@
 	(paper "A4")
 	(title_block
-		(title "Blamp Knob")
-		(date "2026-08-11")
-		(rev "A")
-		(company "VZ")
+		(title "${B_TITLE}")
+		(date "2026-09-13")
+		(rev "${B_REV}")
+		(company "${B_COMPANY}")
 	)
 	(text_box "VDD = 3.3 - 5V"
